File: usb-dmx/pcb/usb-dmx.kicad_pcb (KiCad board)
At the start: 2 copper layers, 25 x 35 mm, 21 parts, among them J1 USB_C_Receptacle_USB2.0_16P, J2 USB_A, SW1 PTS526_SM15_SMTR2_LFS, U1 IP4234CZ6, U2 ADP2108AUJ-3.3, U3 ESP32-S3-MINI-1U, U4 ST485E

Commit message: Adding other Voltage Regulator
Parts:
- added C10: 22uF, Capacitor_SMD:C_0805_2012Metric, F.Cu at (131.3, 98.7)
- added C7: 100nF, Capacitor_SMD:C_0805_2012Metric, F.Cu at (141.1, 85.2)
- added C8: 22uF, Capacitor_SMD:C_0805_2012Metric, F.Cu at (131.3, 94.4)
- added C9: 10uF, Capacitor_SMD:C_0805_2012Metric, F.Cu at (111.4, 101.1)
- added L2: 3u9H, Inductor_SMD:L_0805_2012Metric, F.Cu at (116.4, 84.8)
- added U5: AP63203WU, Package_TO_SOT_SMD:TSOT-23-6, F.Cu at (123.9, 86.0)
