File: pixel-led/pcb/pixel-led.kicad_pcb (KiCad board)
At the start: 2 copper layers, 20 x 44 mm, 22 parts, among them J1 Conn_01x04_Socket, J1 USB_C_Receptacle_USB2.0_16P, J2 USB_A, SW2 SW_Push, U1 AMS1117-3.3, U3 ESP32-S3-MINI-1U, U4 USBLC6-2SC6, U5 MAX485E

Commit message: layouting
Parts:
- removed C6: 0u1F, Capacitor_SMD:C_0603_1608Metric_Pad1.08x0.95mm_HandSolder
- removed the J1 at (133.3, 71.1)
- removed the J1 at (93.6, 56.8)
- removed R1, R2, R5: 5k1, Resistor_SMD:R_0603_1608Metric_Pad0.98x0.95mm_HandSolder
- removed R6: 10k, Resistor_SMD:R_0603_1608Metric_Pad0.98x0.95mm_HandSolder
- removed U5: MAX485E, Package_SO:SOP-8_3.76x4.96mm_P1.27mm
- added J1: Conn_01x04_Socket, Connector_PinHeader_2.54mm:PinHeader_1x04_P2.54mm_Vertical, F.Cu at (108.5, 79.2)
- added U2: TSOP45xx, Package_TO_SOT_THT:TO-92_Inline_Horizontal2, F.Cu at (103.0, 78.5)
- U3: footprint RF_Module:ESP32-S2-MINI-1U -> RF_Module:ESP32-S2-MINI-1
- moved D1 25.4 mm to (97.0, 85.5), turned to -90 degrees
- moved C5 21.1 mm to (108.8, 52.8), turned to 0 degrees
- moved R3 20.6 mm to (100.0, 60.2), turned to 180 degrees
- moved C3 19.0 mm to (96.5, 60.2), turned to 180 degrees
- moved SW2 17.7 mm to (107.5, 57.2), turned to 90 degrees
- moved C1 16.8 mm to (100.0, 58.0)
- moved R4 16.7 mm to (105.8, 52.8), turned to 0 degrees
- moved U1 15.9 mm to (99.2, 53.2)
- moved U4 14.7 mm to (106.9, 49.0), turned to 0 degrees
- moved C4 13.1 mm to (96.8, 80.5), turned to 180 degrees
- moved C7 12.4 mm to (96.8, 78.5), turned to 180 degrees
- moved C2 11.1 mm to (96.5, 58.0), turned to 0 degrees
- moved U3 10.7 mm to (100.0, 69.2), turned to 90 degrees
- moved J2 4.00 mm to (100.0, 36.0)
Connections:
- U3 pad 7: unconnected-(U3-IO3-Pad7) -> IR
Routing:
- net 1: track 29.6 -> 0.00 mm, vias 2 -> 0
- net 2: track 24.9 -> 0.00 mm, vias 2 -> 0
- net 3: track 24.0 -> 0.00 mm, vias 2 -> 0
- net 4: track 23.2 -> 0.00 mm, vias 2 -> 0
- net Net-(U3-EN): track 23.5 -> 4.06 mm, vias 2 -> 0
- net 14: track 13.3 -> 29.4 mm, vias 2 -> 0
- net VCC_5V: track 70.6 -> 86.1 mm
- net GND: track 45.0 -> 30.3 mm, vias 33 -> 35
- net CLK: track 0.00 -> 12.3 mm, vias 0 -> 1
- net DAT: track 0.00 -> 11.5 mm, vias 0 -> 1
- net Net-(J1-D+-PadA6): track 10.4 -> 0.00 mm
- net D-: track 10.0 -> 20.0 mm
- net DMX-: track 9.48 -> 0.00 mm
- net Net-(J2-D-): track 0.00 -> 8.90 mm
- net Net-(J1-D--PadA7): track 8.63 -> 0.00 mm
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Other:
- board size 20 x 44 mm -> 22 x 50 mm
- board text added: "5V"
- board text added: "CLK"
- board text added: "DAT"
- board text added: "GND"
- board text added: "TRANCE PIXEL-LED REV: 1.0"
- board text removed: "${REFERENCE}"
- board text removed: "DESIGNED BY SAMUEL HAFEN"
- board text removed: "TRANCE USB-DMX Rev: 1.2"

Commit message: finishing layout
Parts:
- U2: value TSOP45xx -> TL1838
- moved R4 0.75 mm to (105.7, 52.0)
- moved C5 0.75 mm to (108.8, 52.0)
Connections:
- U2 pad 2: VCC_5V -> GND
- U2 pad 3: GND -> VCC_3.3V
- U3 pad 11: unconnected-(U3-IO7-Pad11) -> CLK
- U3 pad 12: unconnected-(U3-IO8-Pad12) -> DAT
- U3 pad 5: DAT -> unconnected-(U3-IO1-Pad5)
- U3 pad 6: CLK -> unconnected-(U3-IO2-Pad6)
Routing:
- net GND: track 30.3 -> 86.6 mm, vias 35 -> 36
- net VCC_3.3V: track 44.1 -> 59.0 mm
- net 0: track 33.5 -> 40.5 mm
- net DAT: track 11.5 -> 6.79 mm, vias 1 -> 0
- net CLK: track 12.3 -> 9.45 mm, vias 1 -> 0
- net VCC_5V: track 86.1 -> 85.5 mm, vias 2 -> 6
